File: files/Charbdis-Mangleform/main_pcb.kicad_pcb (KiCad board)
At the start: 2 copper layers, 126.3 x 79.2 mm, 82 parts, among them J1 Conn_01x04_Female, J2 Conn_01x05_Female, J3 Conn_01x03_Female, J4 Conn_01x06_Female, J5 Conn_01x03_Female, J7 Conn_01x04, SW10 SW_Push, SW11 SW_Push, SW12 SW_Push, SW15 SW_Push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

Commit message: Update main_pcb.kicad_pcb
Parts:
- D22, D24, D26, D29, D34, D38, D40, D42, D43, D45, D48, D50, D52, D56, D58, D6, D60, D8: moved to B.Cu
- moved D56 203.9 mm to (180.2, 56.6), turned to 180 degrees
- moved D60 192.1 mm to (180.2, 102.6), turned to 180 degrees
- moved D57 181.9 mm to (180.2, 79.7)
- moved D45 181.8 mm to (158.7, 102.6), turned to 180 degrees
- moved D58 181.7 mm to (180.2, 79.7), turned to 180 degrees
- moved D43 169.8 mm to (158.7, 79.7), turned to 180 degrees
- moved D55 164.9 mm to (180.2, 56.6)
- moved D48 156.9 mm to (135.2, 99.0), turned to 180 degrees
- moved D59 155.3 mm to (180.2, 102.6)
- moved D28 153.0 mm to (158.7, 56.7)
- moved D29 151.2 mm to (158.7, 56.7), turned to 180 degrees
- moved D52 148.6 mm to (135.2, 53.3), turned to 180 degrees
- moved D44 144.2 mm to (158.7, 102.6)
- moved D30 141.0 mm to (158.7, 79.7)
- moved D38 139.9 mm to (113.1, 55.2), turned to 180 degrees
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Routing:
- net row1: track 521.3 -> 0.00 mm, vias 8 -> 0
- net row2: track 342.9 -> 263.5 mm
- net col4: track 52.0 -> 0.00 mm
- net col2: track 48.3 -> 0.00 mm
- net col6: track 55.7 -> 7.50 mm, vias 2 -> 0
- net row3: track 509.8 -> 474.0 mm, vias 0 -> 2
- net col1: track 33.1 -> 0.00 mm
- net Net-(D16-Pad2): track 22.3 -> 0.00 mm
- net Net-(D20-Pad2): track 22.1 -> 0.00 mm, vias 2 -> 0
- net Net-(D31-Pad2): track 20.6 -> 0.00 mm, vias 2 -> 0
- net Net-(D15-Pad2): track 20.5 -> 0.00 mm
- net Net-(D17-Pad2): track 20.5 -> 0.00 mm
- net Net-(D36-Pad2): track 19.9 -> 0.00 mm, vias 2 -> 0
- net Net-(D11-Pad2): track 19.1 -> 0.00 mm
- net Net-(D9-Pad2): track 19.0 -> 0.00 mm
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Other:
- board size 126.3 x 79.2 mm -> 126.5 x 90.9 mm

Commit message: routed some more (almost done one side)
Routing:
- net row3: track 474.0 -> 0.00 mm, vias 2 -> 0
- net Net-(D21-Pad2): track 0.00 -> 286.3 mm, vias 0 -> 6
- net row2: track 263.5 -> 0.00 mm
- net Net-(D21-Pad4): track 0.00 -> 148.7 mm, vias 0 -> 4
- net Net-(D41-Pad1): track 0.00 -> 131.1 mm, vias 0 -> 2
- net Net-(D25-Pad1): track 0.00 -> 122.2 mm, vias 0 -> 2
- net Net-(D21-Pad3): track 0.00 -> 119.1 mm
- net Net-(D28-Pad3): track 0.00 -> 101.0 mm, vias 0 -> 2
- net Net-(D28-Pad4): track 0.00 -> 74.7 mm, vias 0 -> 4
- net Net-(D33-Pad4): track 0.00 -> 70.5 mm, vias 0 -> 2
- net row4: track 0.00 -> 58.8 mm
- net col5: track 0.00 -> 58.4 mm, vias 0 -> 3
- net col4: track 0.00 -> 57.7 mm, vias 0 -> 3
- net col6: track 7.50 -> 63.2 mm, vias 0 -> 3
- net Net-(D37-Pad1): track 0.00 -> 50.6 mm
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Other:
- outline, holes or cut-outs redrawn
- board text added: "C1"
- board text removed: "X"
